Commit message: Placing the rplidar on the ros-robot

File: src/learning_nxt/ros_robot4b.urdf (robot description, URDF)
Before this commit: robot ros_robot, 174 links, 173 joints
Links:
- added link laser, mass 1e-5; collision box size=0.001 0.001 0.001; visual mesh filename=package://rplidar_ros/meshes/rplidar-a2m4-r1.stl scale=0.001 0.001 0.001
Joints:
- added joint laser_joint: type fixed, parent ref_125_link, child laser, origin xyz=0 0 0 rpy=0 0 3.14, axis 0 1 0

File: src/ros_robot/ros_robot.urdf (robot description, URDF)
Before this commit: robot ros_robot, 128 links, 127 joints
Links:
- added link laser, mass 1e-5; collision box size=0.001 0.001 0.001; visual mesh filename=package://rplidar_ros/meshes/rplidar-a2m4-r1.stl scale=0.001 0.001 0.001
Joints:
- added joint laser_joint: type fixed, parent ref_0_link, child laser, origin xyz=0.02 0 0.086 rpy=0 0 3.14, axis 0 1 0
