Commit message: Updated urdf model

File: src/ros_robot/ros_robot.urdf (robot description, URDF)
Before this commit: robot ros_robot, 82 links, 81 joints
Links:
- removed link laser_link
- removed link ref_24_link_hub
- removed link ref_31_link
- removed link ref_58_link
- removed link ref_59_link
- removed link ref_60_link
- removed link ref_61_link
- removed link ref_62_link
- removed link ref_63_link
- removed link ref_64_link
- removed link ref_65_link
- removed link ref_66_link
- removed link ref_67_link
- removed link ref_68_link
- removed link ref_69_link
- removed link ref_6_link_hub
- removed link ref_70_link
- removed link ref_71_link
- removed link ref_72_link
- removed link ref_73_link
- removed link ref_74_link
- removed link ref_75_link
- removed link ref_76_link
- removed link ref_77_link
- added link ref_11_link_hub, mass 0.010000; collision box size=0 0 0; visual mesh filename=package://nxt_description/meshes/parts/servo_hubs.dae scale=0.0004 0.0004 0.0004
- added link ref_17_link_hub, mass 0.010000; collision box size=0 0 0; visual mesh filename=package://nxt_description/meshes/parts/servo_hubs.dae scale=0.0004 0.0004 0.0004
- added link ref_38_link, mass 0.010000; collision box size=0 0 0; visual mesh filename=package://nxt_description/meshes/parts/44294.dae scale=0.0004 0.0004 0.0004
- added link ultrasonic_link, mass 0.023900; collision box size=0 0 0; visual mesh filename=package://nxt_description/meshes/parts/53792.dae scale=0.0004 0.0004 0.0004
- link ref_0_link: geometry collision box size=0 0 0; visual mesh filename=package://nxt_description/meshes/parts/2780.dae scale=0.0004 0.0004 0.0004
- link ref_11_link: geometry collision box size=0 0 0; visual mesh filename=package://nxt_description/meshes/parts/53787.dae scale=0.0004 0.0004 0.0004
- link ref_12_link: geometry collision box size=0 0 0; visual mesh filename=package://nxt_description/meshes/parts/2780.dae scale=0.0004 0.0004 0.0004
- link ref_13_link: geometry collision box size=0 0 0; visual mesh filename=package://nxt_description/meshes/parts/2780.dae scale=0.0004 0.0004 0.0004
- link ref_14_link: geometry collision box size=0 0 0; visual mesh filename=package://nxt_description/meshes/parts/40490.dae scale=0.0004 0.0004 0.0004
- link ref_15_link: geometry collision box size=0 0 0; visual mesh filename=package://nxt_description/meshes/parts/2780.dae scale=0.0004 0.0004 0.0004
- link ref_16_link: geometry collision box size=0 0 0; visual mesh filename=package://nxt_description/meshes/parts/2780.dae scale=0.0004 0.0004 0.0004
- link ref_17_link: geometry collision box size=0 0 0; visual mesh filename=package://nxt_description/meshes/parts/53787.dae scale=0.0004 0.0004 0.0004
- link ref_18_link: geometry collision box size=0 0 0; visual mesh filename=package://nxt_description/meshes/parts/32009.dae scale=0.0004 0.0004 0.0004
- link ref_19_link: geometry collision box size=0 0 0; visual mesh filename=package://nxt_description/meshes/parts/3749.dae scale=0.0004 0.0004 0.0004
- link ref_1_link: geometry collision box size=0 0 0; visual mesh filename=package://nxt_description/meshes/parts/53788.dae scale=0.0004 0.0004 0.0004
- link ref_20_link: geometry collision box size=0 0 0; visual mesh filename=package://nxt_description/meshes/parts/3749.dae scale=0.0004 0.0004 0.0004
- link ref_21_link: geometry collision box size=0 0 0; visual mesh filename=package://nxt_description/meshes/parts/2780.dae scale=0.0004 0.0004 0.0004
- link ref_22_link: geometry collision box size=0 0 0; visual mesh filename=package://nxt_description/meshes/parts/6558.dae scale=0.0004 0.0004 0.0004
- link ref_23_link: geometry collision box size=0 0 0; visual mesh filename=package://nxt_description/meshes/parts/41239.dae scale=0.0004 0.0004 0.0004
- link ref_24_link: geometry collision box size=0 0 0; visual mesh filename=package://nxt_description/meshes/parts/6558.dae scale=0.0004 0.0004 0.0004
- link ref_25_link: geometry collision box size=0 0 0; visual mesh filename=package://nxt_description/meshes/parts/41239.dae scale=0.0004 0.0004 0.0004
- link ref_26_link: geometry collision box size=0 0 0; visual mesh filename=package://nxt_description/meshes/parts/6558.dae scale=0.0004 0.0004 0.0004
- link ref_27_link: geometry collision box size=0 0 0; visual mesh filename=package://nxt_description/meshes/parts/32525.dae scale=0.0004 0.0004 0.0004
- link ref_28_link: geometry collision box size=0 0 0; visual mesh filename=package://nxt_description/meshes/parts/6558.dae scale=0.0004 0.0004 0.0004
- link ref_29_link: geometry collision box size=0 0 0; visual mesh filename=package://nxt_description/meshes/parts/32526.dae scale=0.0004 0.0004 0.0004
- link ref_2_link: geometry collision box size=0 0 0; visual mesh filename=package://nxt_description/meshes/parts/2780.dae scale=0.0004 0.0004 0.0004
- link ref_30_link: geometry collision box size=0 0 0; visual mesh filename=package://nxt_description/meshes/parts/6558.dae scale=0.0004 0.0004 0.0004
- link ref_32_link: geometry collision box size=0 0 0; visual mesh filename=package://nxt_description/meshes/parts/6558.dae scale=0.0004 0.0004 0.0004
- link ref_33_link: geometry collision box size=0 0 0; visual mesh filename=package://nxt_description/meshes/parts/32526.dae scale=0.0004 0.0004 0.0004
- link ref_34_link: geometry collision box size=0 0 0; visual mesh filename=package://nxt_description/meshes/parts/6558.dae scale=0.0004 0.0004 0.0004
- link ref_35_link: geometry collision box size=0 0 0; visual mesh filename=package://nxt_description/meshes/parts/32526.dae scale=0.0004 0.0004 0.0004
- link ref_36_link: geometry collision box size=0 0 0; visual mesh filename=package://nxt_description/meshes/parts/6558.dae scale=0.0004 0.0004 0.0004
- link ref_37_link: geometry collision box size=0 0 0; visual mesh filename=package://nxt_description/meshes/parts/6558.dae scale=0.0004 0.0004 0.0004
- link ref_39_link: geometry collision box size=0 0 0; visual mesh filename=package://nxt_description/meshes/parts/3713.dae scale=0.0004 0.0004 0.0004
- link ref_3_link: geometry collision box size=0 0 0; visual mesh filename=package://nxt_description/meshes/parts/32525.dae scale=0.0004 0.0004 0.0004
- link ref_41_link: geometry collision box size=0 0 0; visual mesh filename=package://nxt_description/meshes/parts/32526.dae scale=0.0004 0.0004 0.0004
- link ref_42_link: geometry collision box size=0 0 0; visual mesh filename=package://nxt_description/meshes/parts/6558.dae scale=0.0004 0.0004 0.0004
- link ref_43_link: geometry collision box size=0 0 0; visual mesh filename=package://nxt_description/meshes/parts/6558.dae scale=0.0004 0.0004 0.0004
- link ref_44_link: geometry collision box size=0 0 0; visual mesh filename=package://nxt_description/meshes/parts/6558.dae scale=0.0004 0.0004 0.0004
- link ref_45_link: geometry collision box size=0 0 0; visual mesh filename=package://nxt_description/meshes/parts/6558.dae scale=0.0004 0.0004 0.0004
- link ref_46_link: geometry collision box size=0 0 0; visual mesh filename=package://nxt_description/meshes/parts/6558.dae scale=0.0004 0.0004 0.0004
- link ref_47_link: geometry collision box size=0 0 0; visual mesh filename=package://nxt_description/meshes/parts/41239.dae scale=0.0004 0.0004 0.0004
- link ref_48_link: geometry collision box size=0 0 0; visual mesh filename=package://nxt_description/meshes/parts/6558.dae scale=0.0004 0.0004 0.0004
- link ref_49_link: geometry collision box size=0 0 0; visual mesh filename=package://nxt_description/meshes/parts/32525.dae scale=0.0004 0.0004 0.0004
- link ref_4_link: geometry collision box size=0 0 0; visual mesh filename=package://nxt_description/meshes/parts/2780.dae scale=0.0004 0.0004 0.0004
- link ref_50_link: geometry collision box size=0 0 0; visual mesh filename=package://nxt_description/meshes/parts/2780.dae scale=0.0004 0.0004 0.0004
- link ref_51_link: geometry collision box size=0 0 0; visual mesh filename=package://nxt_description/meshes/parts/32073.dae scale=0.0004 0.0004 0.0004
- link ref_52_link: geometry collision box size=0 0 0; visual mesh filename=package://nxt_description/meshes/parts/56145.dae scale=0.0004 0.0004 0.0004
- link ref_53_link: geometry collision box size=0 0 0; visual mesh filename=package://nxt_description/meshes/parts/44309.dae scale=0.0004 0.0004 0.0004
- link ref_55_link: geometry collision box size=0 0 0; visual mesh filename=package://nxt_description/meshes/parts/44309.dae scale=0.0004 0.0004 0.0004
- link ref_56_link: geometry collision box size=0 0 0; visual mesh filename=package://nxt_description/meshes/parts/56145.dae scale=0.0004 0.0004 0.0004
- link ref_57_link: geometry collision box size=0 0 0; visual mesh filename=package://nxt_description/meshes/parts/32073.dae scale=0.0004 0.0004 0.0004
- link ref_6_link: geometry collision box size=0 0 0; visual mesh filename=package://nxt_description/meshes/parts/41239.dae scale=0.0004 0.0004 0.0004
- link ref_7_link: geometry collision box size=0 0 0; visual mesh filename=package://nxt_description/meshes/parts/6558.dae scale=0.0004 0.0004 0.0004
- link ref_8_link: geometry collision box size=0 0 0; visual mesh filename=package://nxt_description/meshes/parts/32009.dae scale=0.0004 0.0004 0.0004
- link ref_9_link: geometry collision box size=0 0 0; visual mesh filename=package://nxt_description/meshes/parts/3749.dae scale=0.0004 0.0004 0.0004
Joints:
- removed joint ref_58_joint
- removed joint ref_59_joint
- removed joint ref_60_joint
- removed joint ref_61_joint
- removed joint ref_62_joint
- removed joint ref_63_joint
- removed joint ref_64_joint
- removed joint ref_65_joint
- removed joint ref_66_joint
- removed joint ref_67_joint
- removed joint ref_68_joint
- removed joint ref_69_joint
- removed joint ref_70_joint
- removed joint ref_71_joint
- removed joint ref_72_joint
- removed joint ref_73_joint
- removed joint ref_74_joint
- removed joint ref_75_joint
- removed joint ref_76_joint
- removed joint ref_77_joint
- joint base_joint: origin xyz=0.024 0 0.016 rpy=0 0 -1.57079632679 -> xyz=-0.12 0.035 0.070 rpy=0 0 -1.57079633
- joint l_wheel_joint: child ref_24_link_hub -> ref_17_link_hub; parent ref_24_link -> ref_17_link
- joint r_wheel_joint: child ref_6_link_hub -> ref_11_link_hub; parent ref_6_link -> ref_11_link
- joint ref_0_joint: origin xyz=6.1035148974e-09 0.00799965724949 -0.00399998731613 rpy=3.14159265359 1.57079632679 -0.0 -> xyz=0.0359996353149 0.0159995788574 -0.0358009277344 rpy=-0.0 -0.0 -3.14159265359
- joint ref_10_joint: origin xyz=0.056 0.0722 -0.0237999937892 rpy=-1.57079632679 -0.0 1.57079632679 -> xyz=-0.00799999237061 -0.0559999862671 0.00820001422167 rpy=-3.14159265359 -0.0 -0.0; parent ref_5_link -> ref_7_link
- joint ref_11_joint: origin xyz=0.016 0.040000012207 -0.0240000037193 rpy=-0.0 -0.0 -1.57079632679 -> xyz=-0.0161999929547 0.000199948120117 -0.00399998779297 rpy=1.57079632679 -1.57079632679 -0.0; parent ref_5_link -> ref_8_link
- joint ref_12_joint: origin xyz=0.062 0.040000012207 -0.0240000037193 rpy=-0.0 -0.0 1.57079632679 -> xyz=-0.00420001398325 -0.00779998931885 -0.0239999664307 rpy=-1.57079632679 -0.0 -3.14159265359; parent ref_5_link -> ref_8_link
- joint ref_13_joint: origin xyz=-0.0300000244141 0.040000012207 -0.0239999987602 rpy=-0.0 -0.0 1.57079632679 -> xyz=-0.00399999923706 0.0159999941826 -3.0517578125e-09 rpy=3.14159265359 1.57079632679 -0.0; parent ref_5_link -> ref_13_link
- joint ref_14_joint: origin xyz=-0.008 0.0800000061035 -0.0240000052452 rpy=0.0 1.57079632679 -0.0 -> xyz=-0.0 0.0319999991417 -0.00399999923706 rpy=3.14159265359 1.57079632679 -0.0; parent ref_5_link -> ref_14_link
- joint ref_15_joint: origin xyz=1.220703125e-08 0.0800000061035 -0.0240500037223 rpy=-1.57079632679 1.57079632679 -0.0 -> xyz=-6.103515625e-09 -0.0160000052452 -0.00399999923706 rpy=3.14159265359 1.57079632679 -0.0; parent ref_5_link -> ref_14_link
- joint ref_16_joint: origin xyz=0.00800001220703 0.0800000061035 -0.0240000052452 rpy=0.0 1.57079632679 -0.0 -> xyz=0.0839999755859 0.00800001068115 0.000200012207031 rpy=-3.14159265359 -0.0 1.57079632679; parent ref_5_link -> ref_16_link
- joint ref_17_joint: origin xyz=1.220703125e-08 0.104 -0.0240500037223 rpy=-1.57079632679 1.57079632679 -0.0 -> xyz=-0.00419999923706 0.0240000228882 -0.007800050354 rpy=-1.57079632679 -0.0 -3.14159265359; parent ref_5_link -> ref_16_link
- joint ref_18_joint: origin xyz=0.016 0.072 -0.0240500037223 rpy=-1.57079632679 1.57079632679 -0.0 -> xyz=-0.00399999694824 0.0200000045776 0.0559999969482 rpy=-0.0 -0.0 -1.57079632679; parent ref_5_link -> ref_16_link
- joint ref_19_joint: origin xyz=0.023999987793 0.0800000061035 -0.0240000052452 rpy=0.0 1.57079632679 -0.0 -> xyz=0.0279999847412 0.0200000045776 -0.00799999694824 rpy=-0.0 -0.0 -1.57079632679; parent ref_5_link -> ref_16_link
- joint ref_1_joint: origin xyz=0.004 -0.00020029296875 0.0002 rpy=3.14159265359 -1.57079632679 -0.0 -> xyz=-0.0360000289917 0.0160000152588 0.0197999950767 rpy=-0.0 -0.0 -3.14159265359
- joint ref_20_joint: origin xyz=0.032 0.0800000061035 -0.0240500037223 rpy=-1.57079632679 1.57079632679 -0.0 -> xyz=0.0119999969482 -0.0719999832153 0.00820000915527 rpy=-3.14159265359 -0.0 -3.14159265359; parent ref_5_link -> ref_17_link
- joint ref_21_joint: origin xyz=0.04 0.0800000061035 -0.0240000052452 rpy=0.0 1.57079632679 -0.0 -> xyz=-0.00800000610352 -0.0559999694824 0.00820001373291 rpy=-3.14159265359 -0.0 -3.14159265359; parent ref_5_link -> ref_17_link
- joint ref_22_joint: origin xyz=0.032 0.104 -0.0240500037223 rpy=-1.57079632679 1.57079632679 -0.0 -> xyz=0.00800000076294 -0.0480000183105 -0.0 rpy=3.14159265359 1.57079632679 -0.0; parent ref_5_link -> ref_22_link
- joint ref_23_joint: origin xyz=-0.00799997558594 -0.0159999755859 -0.0157999894977 rpy=-3.14159265359 -0.0 -0.0 -> xyz=-0.0 0.0159999980927 -0.00799998092652 rpy=0.0 -1.57079632679 -0.0; parent ref_5_link -> ref_23_link
- joint ref_24_joint: origin xyz=0.00799998779297 2.44140625e-08 0.000200012969971 rpy=-3.14159265359 -0.0 -3.14159265359 -> xyz=-0.00800000286102 -0.016 -0.0 rpy=0.0 1.57079632679 -0.0; parent ref_6_link -> ref_24_link
- joint ref_25_joint: origin xyz=0.023199987793 2.44140625e-08 1.14440917969e-08 rpy=-1.57079632679 -1.57079632679 -0.0 -> xyz=-0.0 -0.0239999975204 0.00800000190735 rpy=0.0 -1.57079632679 -0.0; parent ref_6_link -> ref_25_link
- joint ref_26_joint: origin xyz=0.023199987793 2.44140625e-08 1.14440917969e-08 rpy=-3.14159265359 -0.0 -1.57079632679 -> xyz=5.66244125366e-09 -0.031999993515 -0.0 rpy=0.0 1.57079632679 -0.0; parent ref_6_link -> ref_26_link
- joint ref_27_joint: origin xyz=-0.055999987793 2.44140625e-08 0.000200012969971 rpy=-3.14159265359 -0.0 -3.14159265359 -> xyz=-0.0 -0.0160000072479 1.49011594175e-09 rpy=0.0 -1.57079632679 -0.0; parent ref_6_link -> ref_27_link
- joint ref_28_joint: origin xyz=-0.068 2.44140625e-08 1.14440917969e-08 rpy=1.57079632679 -1.57079632679 -0.0 -> xyz=0.00799999685287 0.000200006103516 0.0322000003934 rpy=-1.57079632679 -0.0 1.57079632679; parent ref_6_link -> ref_28_link
- joint ref_29_joint: origin xyz=-0.068 2.44140625e-08 1.14440917969e-08 rpy=-3.14159265359 -0.0 1.57079632679 -> xyz=-0.000200006115437 0.0002 0.00799999446869 rpy=1.57079632679 1.57079632679 -0.0; parent ref_6_link -> ref_29_link
- joint ref_2_joint: origin xyz=0.00779999907017 0.0157999981165 0.00799999904633 rpy=0.0 1.57079632679 -0.0 -> xyz=0.00400000305176 -0.000199996948242 -0.023799987793 rpy=-1.57079632679 -0.0 -1.57079632679
- joint ref_30_joint: child ref_31_link -> ultrasonic_link; origin xyz=-0.0439999755859 -0.00799997558594 -0.0157999885559 rpy=-3.14159265359 -0.0 -3.14159265359 -> xyz=-5.06639480591e-09 -0.00799999694824 0.000200000011921 rpy=-0.0 -0.0 -0.0; parent ref_6_link -> ref_30_link
- joint ref_31_joint: origin xyz=-0.00399998779297 0.015999987793 -0.0 rpy=3.14159265359 1.57079632679 -0.0 -> xyz=-8.94069671631e-10 -6.103515625e-09 -0.000200000011921 rpy=-0.0 -0.0 -0.0; parent ref_31_link -> ultrasonic_link
- joint ref_32_joint: origin xyz=6.1035148974e-09 0.00799968166355 0.00400001173019 rpy=3.14159265359 1.57079632679 -0.0 -> xyz=0.00800000424385 -0.0161999938965 -0.0318000003695 rpy=1.57079632679 -0.0 -1.57079632679
- joint ref_33_joint: origin xyz=-0.0 0.0319999839783 -0.00399998731613 rpy=3.14159265359 1.57079632679 -0.0 -> xyz=-0.0002 0.00779999754429 0.0079999997139 rpy=-1.57079632679 1.57079632679 -0.0; parent ref_32_link -> ref_33_link
- joint ref_34_joint: origin xyz=-0.0 -0.0079999868393 0.0159999858856 rpy=3.14159265359 1.57079632679 -0.0 -> xyz=-0.00800000238419 -0.0002 -0.00779999893904 rpy=1.57079632679 -0.0 -1.57079632679; parent ref_32_link -> ref_34_link
- joint ref_35_joint: origin xyz=-0.0 -0.0079999868393 0.0239999849319 rpy=1.57079632679 -0.0 -1.57079632679 -> xyz=-0.0082 0.0317999946833 -0.00799999666214 rpy=-1.57079632679 1.57079632679 -0.0; parent ref_32_link -> ref_35_link
- joint ref_36_joint: origin xyz=-0.0 -0.0079999868393 0.00799999904633 rpy=1.57079632679 -0.0 -1.57079632679 -> xyz=-0.0002 -0.000199999976158 -0.00799999666214 rpy=-1.57079632679 1.57079632679 -0.0; parent ref_32_link -> ref_35_link
- joint ref_37_joint: child laser_link -> ref_38_link; origin xyz=-0.0 0.00799997558594 0.0002 rpy=-3.14159265359 -0.0 -0.0 -> xyz=-0.000200006103516 0.0237999925852 -0.00800000143051 rpy=-1.57079632679 -1.57079632679 -0.0
- joint ref_38_joint: origin xyz=-0.0 -0.00800003566742 0.0002 rpy=-3.14159265359 -0.0 -0.0 -> xyz=-0.000199993896484 0.0237999925852 0.00800000591278 rpy=-1.57079632679 -0.0 -0.0; parent laser_link -> ref_35_link
- joint ref_39_joint: origin xyz=-0.00799999904633 -0.00800003566742 0.0002 rpy=-3.14159265359 -0.0 -1.57079632679 -> xyz=-0.000199993896484 0.0237999925852 -0.0239999933243 rpy=-1.57079632679 -0.0 -0.0; parent laser_link -> ref_35_link
- joint ref_3_joint: origin xyz=-0.008 -0.0158 -0.00780000046492 rpy=0.0 -1.57079632679 -0.0 -> xyz=-0.000199990856647 -0.0397999816895 -0.00400000305176 rpy=1.57079632679 -1.57079632679 -0.0
- joint ref_40_joint: child ref_41_link -> color_link; origin xyz=0.0079999868393 -0.00800003566742 0.0002 rpy=-3.14159265359 -0.0 -1.57079632679 -> xyz=4.17232513428e-10 6.103515625e-09 -0.00780000305176 rpy=1.57079632679 -0.0 -3.14159265359; parent laser_link -> ref_38_link
- joint ref_41_joint: child ref_42_link -> ref_41_link; origin xyz=-0.0078 -0.127999981689 0.00400001449585 rpy=0.0 -1.57079632679 -0.0 -> xyz=-0.00800000019073 0.000200006103516 0.000200000011921 rpy=-1.57079632679 -0.0 1.57079632679; parent ref_6_link -> ref_30_link
- joint ref_42_joint: child ref_43_link -> ref_42_link; origin xyz=-0.00399952573782 -0.000200027441975 0.0161998393774 rpy=-1.57079632679 -0.0 -1.57079632679 -> xyz=-0.0161999979138 0.0321999984741 -0.00799999780655 rpy=1.57079632679 1.57079632679 -0.0; parent ref_42_link -> ref_41_link
- joint ref_43_joint: child ref_44_link -> ref_43_link; origin xyz=-0.000200283813477 0.0321997558594 0.003999193573 rpy=1.57079632679 -1.57079632679 -0.0 -> xyz=-0.0 0.0399999883652 -8.94069565049e-10 rpy=0.0 -1.57079632679 -0.0; parent ref_43_link -> ref_27_link
- joint ref_44_joint: child ref_45_link -> ref_44_link; origin xyz=-0.000199987792969 -0.031799987793 0.00399999847412 rpy=1.57079632679 -1.57079632679 -0.0 -> xyz=-0.0 0.0159999874115 -5.66244057865e-09 rpy=0.0 -1.57079632679 -0.0; parent ref_43_link -> ref_27_link
- joint ref_45_joint: child ref_46_link -> ref_45_link; origin xyz=-0.000199978637695 0.0002 0.00399999694824 rpy=1.57079632679 -1.57079632679 -0.0 -> xyz=-0.0 -0.0319999984741 -0.00799999828339 rpy=0.0 -1.57079632679 -0.0; parent ref_43_link -> ref_25_link
- joint ref_46_joint: child ref_47_link -> ref_46_link; origin xyz=-0.00020002746582 -0.0158001342773 0.0039995262146 rpy=1.57079632679 -1.57079632679 -0.0 -> xyz=-1.52587872435e-09 -0.0320000007629 0.00799999828339 rpy=3.14159265359 1.57079632679 -0.0; parent ref_43_link -> ref_23_link
- joint ref_47_joint: child ref_48_link -> ref_47_link; origin xyz=-0.0519997802734 -0.136000302124 0.00820084648132 rpy=-3.14159265359 -0.0 -3.14159265359 -> xyz=-0.00800000610352 -0.0319999954224 -1.5258789972e-09 rpy=3.14159265359 1.57079632679 -0.0; parent ref_6_link -> ref_46_link
- joint ref_48_joint: child ref_49_link -> ref_48_link; origin xyz=0.004 -0.135999865723 0.0081999080658 rpy=-3.14159265359 -0.0 -3.14159265359 -> xyz=-0.0 0.0159999919891 0.00799999446869 rpy=0.0 -1.57079632679 -0.0; parent ref_6_link -> ref_47_link
- joint ref_49_joint: child ref_50_link -> ref_49_link; origin xyz=-0.055999987793 -0.119800140381 0.00800017471313 rpy=-1.57079632679 -0.0 -3.14159265359 -> xyz=0.00799967346191 0.000199728393555 0.0402007760168 rpy=-1.57079632679 -0.0 1.57079632679; parent ref_6_link -> ref_48_link
- joint ref_4_joint: origin xyz=-0.000199993872643 0.0158000103235 0.00800001125336 rpy=0.0 1.57079632679 -0.0 -> xyz=-0.000200161755095 0.0401998336792 -0.00799999389648 rpy=1.57079632679 1.57079632679 -0.0; parent ref_4_link -> ref_3_link
- joint ref_50_joint: child ref_51_link -> ref_50_link; origin xyz=0.00800001125336 0.039999990654 0.000399999952316 rpy=3.14159265359 -1.57079632679 -0.0 -> xyz=-0.000199990856647 -0.023799987793 0.00399999694824 rpy=1.57079632679 -1.57079632679 -0.0; parent ref_50_link -> ref_49_link
- joint ref_51_joint: child ref_52_link -> ref_51_link; origin xyz=-0.000199993908405 -0.0237999969482 -0.00400001220703 rpy=1.57079632679 -1.57079632679 -0.0 -> xyz=0.00799998474121 1.8310546875e-08 0.000200012207031 rpy=-3.14159265359 -0.0 -3.14159265359; parent ref_51_link -> ref_17_link
- joint ref_52_joint: child ref_53_link -> ref_52_link; origin xyz=-0.0360000244141 0.0160000183105 -0.0198000030518 rpy=-0.0 -0.0 -3.14159265359 -> xyz=0.019999987793 2.44140625e-08 1.220703125e-08 rpy=-1.57079632679 -1.57079632679 -0.0; parent ref_52_link -> ref_17_link
- joint ref_53_joint: child ref_54_link -> ref_53_link; origin xyz=0.0359996337891 0.0159995849609 0.0198009380699 rpy=-0.0 -0.0 -3.14159265359 -> xyz=0.019499987793 2.44140625e-08 1.220703125e-08 rpy=-3.14159265359 -0.0 -1.57079632679; parent ref_53_link -> ref_17_link
- joint ref_54_joint: child ref_55_link -> ref_54_link; origin xyz=-0.004 -0.000199987792969 -0.0237999938965 rpy=-1.57079632679 -0.0 -1.57079632679 -> xyz=0.00799999389648 -0.0839999664307 0.000200012207031 rpy=-3.14159265359 -0.0 1.57079632679; parent ref_54_link -> ref_17_link
- joint ref_55_joint: child ref_56_link -> ref_55_link; origin xyz=-0.000399938988682 0.0400000488281 0.008 rpy=2.37436070984 -1.57077705027 0.758112229805 -> xyz=-0.08820001899 -0.00799999237061 0.0053000213623 rpy=1.57079632679 -0.0 -0.0; parent ref_55_link -> ref_8_link
- joint ref_56_joint: child ref_57_link -> ref_56_link; origin xyz=-0.000199993908405 -0.0397999816895 0.004 rpy=1.57079632679 -1.57079632679 -0.0 -> xyz=-0.08820001899 -0.00799999237061 0.0048000213623 rpy=1.57079632679 -0.0 1.57079632679; parent ref_55_link -> ref_8_link
- joint ref_57_joint: child ref_58_link -> ref_57_link; origin xyz=-0.0360000244141 0.0160000244141 0.0357999929786 rpy=-0.0 -0.0 -3.14159265359 -> xyz=-0.0882000128865 -0.00779999237061 -0.00799998474121 rpy=1.57079632679 -1.57079632679 -0.0; parent ref_53_link -> ref_8_link
- joint ref_5_joint: origin xyz=0.04 -0.0159999755859 -0.0157999894977 rpy=-3.14159265359 -0.0 -0.0 -> xyz=0.00800000915527 -0.016 -0.0 rpy=0.0 1.57079632679 -0.0
- joint ref_6_joint: origin xyz=-0.0239999755859 0.0722000183105 -0.0237999937892 rpy=-1.57079632679 -0.0 1.57079632679 -> xyz=-0.0 -0.0479999866486 0.00800000209808 rpy=0.0 -1.57079632679 -0.0; parent ref_5_link -> ref_6_link
- joint ref_7_joint: origin xyz=-0.019999987793 0.0720000183105 0.0400000023842 rpy=-0.0 -0.0 -0.0 -> xyz=-0.0239999847412 0.0322000030518 0.000200009167195 rpy=-1.57079632679 -0.0 1.57079632679; parent ref_5_link -> ref_7_link
- joint ref_8_joint: origin xyz=0.016 0.0400000244141 -0.0240000037193 rpy=-0.0 -0.0 -3.14159265359 -> xyz=-0.0199999908447 0.0320000007629 0.0640000022888 rpy=-0.0 -0.0 -0.0; parent ref_5_link -> ref_7_link
- joint ref_9_joint: origin xyz=0.052 0.072 0.0400000023842 rpy=-0.0 -0.0 -3.14159265359 -> xyz=-0.02 1.220703125e-08 6.1035159888e-08 rpy=-0.0 -0.0 -0.0; parent ref_5_link -> ref_7_link
