Commit message: Added map

File: src/ros_robot/ros_robot.urdf (robot description, URDF)
Before this commit: robot nxt_ros_robot, 62 links, 61 joints
Joints:
- joint ref_30_joint: origin xyz=-5.06639480591e-09 -0.00799999694824 0.000200000011921 rpy=-0.0 -0.0 -0.0 -> xyz=-4.06639480591e-09 -0.00799999694824 0.000200000011921 rpy=-0.0 -0.0 -0.0

Commit message: new maps

File: src/ros_robot/ros_robot.urdf (robot description, URDF)
Before this commit: robot ros_robot, 5 links, 4 joints
Joints:
- joint l_wheel_joint: axis 1 0 0 -> 0 0 1
- joint r_wheel_joint: axis 1 0 0 -> 0 0 1

Commit message: new rviz conf and use of base_footprint

File: src/ros_robot/ros_robot.urdf (robot description, URDF)
Before this commit: robot ros_robot, 5 links, 4 joints
Links:
- removed link body_frame
- added link base_footprint
- link base_link: geometry visual box size=0.25 0.14 0.10
Joints:
- removed joint body_joint
- added joint base_joint: type fixed, parent base_footprint, child base_link, origin xyz=0 0 0.0779 rpy=0 0 0
- joint l_wheel_joint: parent body_frame -> base_link
- joint laser_joint: parent body_frame -> base_link
- joint r_wheel_joint: parent body_frame -> base_link

Commit message: Config updates

File: src/ros_robot/ros_robot.urdf (robot description, URDF)
Before this commit: robot ros_robot, 5 links, 4 joints
Links:
- link base_link: geometry visual box size=0.25 0.12 0.10
- link l_wheel_frame: geometry visual cylinder length=0.025 radius=0.028
- link r_wheel_frame: geometry visual cylinder length=0.025 radius=0.028
Joints:
- joint l_wheel_joint: origin xyz=0 0.07 -0.0578 rpy=1.5707963268 0 0 -> xyz=0 0.0625 -0.05 rpy=1.5707963268 0 0
- joint laser_joint: origin xyz=0 0 0.07 rpy=0 0 0 -> xyz=0 0 0.06 rpy=0 0 0
- joint r_wheel_joint: origin xyz=0 -0.07 -0.0578 rpy=1.5707963268 0 0 -> xyz=0 -0.0625 -0.05 rpy=1.5707963268 0 0
